File: HW/IsolatedThreeOutputSMPS/ExternRegulatedConverters/ExternRegulatedConverter_5D_12S_5S/ExternRegulatedConverter.kicad_pcb (KiCad board)
At the start: 2 copper layers, 71.1 x 49.5 mm, 20 parts, among them J1 15VDC, U1 MEA1D1505DC, U2 LM7805_TO220, U5 LM7812_TO220

Commit message: update
Parts:
- moved C1 2.80 mm to (117.1, 94.1)
Routing:
- net Net-(C1-Pad1): track 20.3 -> 17.6 mm
- net +15V: track 86.4 -> 89.1 mm
- net GNDA: track 157.0 -> 158.6 mm
