File: HW/CurrentSinkModule/CurrentSinkModule/CurrentSink.sch (KiCad schematic (older format))
At the start: 105 parts, among them J1 Conn_01x03, J2 Conn_01x03, J3 MosfetSocketx3, J4 MosfetSocketx3, U1 LTC2058, U2 LTC2058, U3 LTC2058, U4 LTC2058

Commit message: current module hw update
- Deleted opamp Bypass jumpers in schematic; they break opamp configurations
- Added bypass instructions in schematic for each opamp.
Parts:
- removed JP10, JP5, JP6, JP7, JP8, JP9: BYPASS, Jumper:SolderJumper-2_P1.3mm_Open_Pad1.0x1.5mm, symbol Device:Jumper_NO_Small
Other:
- note added: "INPUT BIAS COMPENSATION.\nIF NOT USED MUST \nBE POPULATED WITH 0R RESISTOR"
- note added: "To bypass active filter populate:\nR1, R3 and R19 with 0R resistors,\nomit others"
- note added: "To bypass active filter populate:\nR2, R4 and R20 with 0R resistors,\nomit others"
- note added: "To bypass inverting gain amp populate:\nR7 and R8 with 1K resistors, R5 with 0R resistor,\nomit others"
- note added: "To bypass inverting opamp populate:\nR13 and R16 with 1K resistors, R22 0R,\nomit others"
- note added: "To bypass non-inverting \ngain amp populate:\nR25 and R6 with 0R resistors\nomit others"
- note added: "To bypass non-inverting opamp populate:\nR14 and R23 with 0R resistors,\nomit others"
Changed lines of the file:
@@
 Wire Wire Line
 	25100 8000 25100 7250
-Wire Wire Line
-	25100 7250 25350 7250
 $Comp
 L Device:R R14
@@
 	0    1    1    0
 $EndComp
-Wire Wire Line
-	23000 7150 22600 7150
 Connection ~ 21950 7150
 Wire Wire Line
@@
 	0    1    1    0
 $EndComp
-Wire Wire Line
-	21950 14200 22225 14200
 Connection ~ 21950 14200
 Wire Wire Line
@@
 Text Label 2575 6300 0    50   ~ 0
 DACSIG1
-Wire Wire Line
-	6000 6400 6300 6400
 $Comp
 L Device:C C2
@@
 	1    0    0    -1
 $EndComp
-Wire Wire Line
-	6250 15300 6550 15300
 $Comp
 L Device:C C1
@@
 Wire Wire Line
 	13250 15325 14400 15325
-$Comp
-L Device:Jumper_NO_Small JP5
-U 1 1 5D41CFB9
-P 5975 14750
-F 0 "JP5" H 5975 14935 50  0000 C CNN
-F 1 "BYPASS" H 5975 14844 50  0000 C CNN
-F 2 "Jumper:SolderJumper-2_P1.3mm_Open_Pad1.0x1.5mm" H 5975 14750 50  0001 C CNN
-F 3 "~" H 5975 14750 50  0001 C CNN
-	1    5975 14750
-	1    0    0    -1
-$EndComp
-Wire Wire Line
-	5875 14750 5300 14750
-Wire Wire Line
-	6075 14750 6550 14750
-Wire Wire Line
-	6550 14750 6550 15300
-Connection ~ 6550 15300
-Wire Wire Line
-	6550 15300 6800 15300
-Wire Wire Line
-	5300 15200 5300 14750
-Connection ~ 5300 15200
-Wire Wire Line
-	5300 15200 5650 15200
-$Comp
-L Device:Jumper_NO_Small JP6
-U 1 1 5D4EBEF2
-P 5725 5850
-F 0 "JP6" H 5725 6035 50  0000 C CNN
-F 1 "BYPASS" H 5725 5944 50  0000 C CNN
-F 2 "Jumper:SolderJumper-2_P1.3mm_Open_Pad1.0x1.5mm" H 5725 5850 50  0001 C CNN
-F 3 "~" H 5725 5850 50  0001 C CNN
-	1    5725 5850
-	1    0    0    -1
-$EndComp
-Wire Wire Line
-	5625 5850 5050 5850
-Wire Wire Line
-	5825 5850 6300 5850
-Wire Wire Line
-	6300 5850 6300 6400
-Wire Wire Line
-	5050 6300 5050 5850
-Connection ~ 5050 6300
-Wire Wire Line
-	5050 6300 5400 6300
-Connection ~ 6300 6400
-Wire Wire Line
-	6300 6400 6600 6400
 $Comp
 L Connector:TestPoint TP3
@@
 Text Notes 24350 8275 2    50   ~ 0
 INPUT BIAS\nCOMPENSATION
-Text Notes 13225 5850 2    50   ~ 0
-INPUT BIAS\nCOMPENSATION
+Text Notes 12500 6000 0    50   ~ 0
+INPUT BIAS COMPENSATION.\nIF NOT USED MUST \nBE POPULATED WITH 0R RESISTOR
 Text Notes 13325 15600 2    50   ~ 0
 INPUT BIAS\nCOMPENSATION
@@
 Connection ~ 4850 15200
 Wire Wire Line
-	4850 15200 5300 15200
-Wire Wire Line
 	4850 15800 4850 15975
 $Comp
@@
 	4750 6575 4750 6300
 Connection ~ 4750 6300
-Wire Wire Line
-	4750 6300 5050 6300
 Wire Wire Line
 	4750 6875 4750 7075
@@
 Wire Wire Line
 	6600 6400 6600 7150
-$Comp
-L Device:Jumper_NO_Small JP8
-U 1 1 5D792CA6
-P 9200 7825
-F 0 "JP8" H 9200 8010 50  0000 C CNN
-F 1 "BYPASS" H 9200 7919 50  0000 C CNN
-F 2 "Jumper:SolderJumper-2_P1.3mm_Open_Pad1.0x1.5mm" H 9200 7825 50  0001 C CNN
-F 3 "~" H 9200 7825 50  0001 C CNN
-	1    9200 7825
-	1    0    0    1
-$EndComp
-Wire Wire Line
-	9100 7825 8375 7825
-Wire Wire Line
-	9300 7825 9775 7825
-Wire Wire Line
-	9775 7825 9775 7250
-Wire Wire Line
-	8375 7250 8375 7825
 Wire Wire Line
 	10300 3900 10300 6500
@@
 ADCSIG2
 Wire Wire Line
-	25650 14300 25875 14300
-Wire Wire Line
 	25650 14300 25100 14300
 Connection ~ 25650 14300
@@
 Wire Wire Line
 	9425 16025 10250 16025
-$Comp
-L Device:Jumper_NO_Small JP7
-U 1 1 5DB4E932
-P 8850 14850
-F 0 "JP7" H 8850 15035 50  0000 C CNN
-F 1 "BYPASS" H 8850 14944 50  0000 C CNN
-F 2 "Jumper:SolderJumper-2_P1.3mm_Open_Pad1.0x1.5mm" H 8850 14850 50  0001 C CNN
-F 3 "~" H 8850 14850 50  0001 C CNN
-	1    8850 14850
-	1    0    0    -1
-$EndComp
-Wire Wire Line
-	8750 14850 8025 14850
-Wire Wire Line
-	8950 14850 9425 14850
-Wire Wire Line
-	9425 14850 9425 15400
-Wire Wire Line
-	8025 15300 8025 14850
 Connection ~ 8025 15300
 Wire Wire Line
@@
 	9425 15400 9425 16025
 Wire Wire Line
-	8025 14850 8025 14350
-Wire Wire Line
 	8025 14350 8600 14350
-Connection ~ 8025 14850
 Wire Wire Line
 	8900 14350 9425 14350
-Wire Wire Line
-	9425 14350 9425 14850
-Connection ~ 9425 14850
 Wire Wire Line
 	7625 6400 7950 6400
@@
 Wire Wire Line
 	7950 6400 8675 6400
-Connection ~ 9775 7250
-Connection ~ 8375 7250
 $Comp
 L power:+12V #PWR0107
@@
 	-1   0    0    1
 $EndComp
-$Comp
-L Device:Jumper_NO_Small JP10
-U 1 1 5D36180C
-P 24175 6275
-F 0 "JP10" H 24175 6460 50  0000 C CNN
-F 1 "BYPASS" H 24175 6369 50  0000 C CNN
-F 2 "Jumper:SolderJumper-2_P1.3mm_Open_Pad1.0x1.5mm" H 24175 6275 50  0001 C CNN
-F 3 "~" H 24175 6275 50  0001 C CNN
-	1    24175 6275
-	1    0    0    1
-$EndComp
-Wire Wire Line
-	24075 6275 22600 6275
-Wire Wire Line
-	22600 6275 22600 7150
-Connection ~ 22600 7150
-Wire Wire Line
-	22600 7150 21950 7150
-Wire Wire Line
-	24275 6275 25350 6275
-Wire Wire Line
-	25350 6275 25350 7250
-Connection ~ 25350 7250
-Wire Wire Line
-	25350 7250 25600 7250
-$Comp
-L Device:Jumper_NO_Small JP9
-U 1 1 5D3A9422
-P 24075 13300
-F 0 "JP9" H 24075 13485 50  0000 C CNN
-F 1 "BYPASS" H 24075 13394 50  0000 C CNN
-F 2 "Jumper:SolderJumper-2_P1.3mm_Open_Pad1.0x1.5mm" H 24075 13300 50  0001 C CNN
-F 3 "~" H 24075 13300 50  0001 C CNN
-	1    24075 13300
-	1    0    0    1
-$EndComp
-Wire Wire Line
-	23975 13300 22225 13300
-Wire Wire Line
-	22225 13300 22225 14200
-Connection ~ 22225 14200
-Wire Wire Line
-	22225 14200 22500 14200
-Wire Wire Line
-	24175 13300 25875 13300
-Wire Wire Line
-	25875 13300 25875 14300
-Connection ~ 25875 14300
-Wire Wire Line
-	25875 14300 26150 14300
+Wire Wire Line
+	6000 6400 6600 6400
+Wire Wire Line
+	4750 6300 5400 6300
+Text Notes 3800 4450 0    100  ~ 0
+To bypass active filter populate:\nR2, R4 and R20 with 0R resistors,\nomit others
+Wire Wire Line
+	6250 15300 6800 15300
+Wire Wire Line
+	4850 15200 5650 15200
+Wire Wire Line
+	8025 14350 8025 15300
+Wire Wire Line
+	9425 14350 9425 15400
+Text Notes 4000 13300 0    100  ~ 0
+To bypass active filter populate:\nR1, R3 and R19 with 0R resistors,\nomit others
+Text Notes 7500 13300 0    100  ~ 0
+To bypass inverting gain amp populate:\nR7 and R8 with 1K resistors, R5 with 0R resistor,\nomit others
+Text Notes 7050 4550 0    100  ~ 0
+To bypass non-inverting \ngain amp populate:\nR25 and R6 with 0R resistors\nomit others
+Text Notes 23400 5900 0    100  ~ 0
+To bypass non-inverting opamp populate:\nR14 and R23 with 0R resistors,\nomit others
+Wire Wire Line
+	21950 7150 23000 7150
+Wire Wire Line
+	25100 7250 25600 7250
+Wire Wire Line
+	21950 14200 22500 14200
+Wire Wire Line
+	25650 14300 26150 14300
+Text Notes 23250 13650 0    100  ~ 0
+To bypass inverting opamp populate:\nR13 and R16 with 1K resistors, R22 0R,\nomit others
 $EndSCHEMATC

Commit message: added notes to current sink module schematic
Other:
- note added: "Expect increasing negative voltage on TP10 and TP12 as U4A output voltage increases. \nTP9 should remain at GND (some offset normal).\nThe output is inverted by U4B so TP14 should increase inversely proportional to TP10 and TP12."
- note added: "Expect increasing positive voltage on TP8 and TP11 as U3A output voltage increases. \nTP7 should remain at GND (some offset normal)."
- note added: "N-Channel\nPower Mosfet"
- note added: "P-Channel\nPower Mosfet"
- note removed: "Power Mosfet"
Changed lines of the file:
@@
 Connection ~ 20450 14850
 Wire Wire Line
-	20450 14850 20450 16100
+	20450 14850 20450 15450
 Wire Wire Line
 	20450 14850 20700 14850
@@
 Text Label 28900 8650 2    50   ~ 0
 DUT_POS
-Text Notes 14500 6150 0    50   ~ 0
-Power Mosfet
+Text Notes 14650 5050 0    50   ~ 0
+N-Channel\nPower Mosfet
 Text Notes 13675 7225 0    50   ~ 0
 Power Resistor\nArcol HS100 \n1ohm 100W
-Text Notes 14475 15175 0    50   ~ 0
-Power Mosfet
+Text Notes 14750 15650 0    50   ~ 0
+P-Channel\nPower Mosfet
 Text Notes 19700 6750 0    50   ~ 0
 InstGain: 14dB
@@
 U 1 1 5D4094FF
 P 14600 15925
-F 0 "J4" H 14518 15600 50  0000 C CNN
-F 1 "MosfetSocketx3" H 14518 15691 50  0000 C CNN
+F 0 "J4" H 14800 15850 50  0000 C CNN
+F 1 "MosfetSocketx3" H 15000 16000 50  0000 C CNN
 F 2 "TerminalBlock:TerminalBlock_bornier-3_P5.08mm" H 14600 15925 50  0001 C CNN
 F 3 "https://docs-emea.rs-online.com/webdocs/0130/0900766b8013040c.pdf" H 14600 15925 50  0001 C CNN
@@
 L power:-12V #PWR0117
 U 1 1 5D72B6A4
-P 20450 16100
-F 0 "#PWR0117" H 20450 16200 50  0001 C CNN
-F 1 "-12V" H 20465 16271 50  0000 C CNN
-F 2 "" H 20450 16100 50  0001 C CNN
-F 3 "" H 20450 16100 50  0001 C CNN
-	1    20450 16100
+P 20450 15450
+F 0 "#PWR0117" H 20450 15550 50  0001 C CNN
+F 1 "-12V" H 20465 15621 50  0000 C CNN
+F 2 "" H 20450 15450 50  0001 C CNN
+F 3 "" H 20450 15450 50  0001 C CNN
+	1    20450 15450
 	-1   0    0    1
 $EndComp
@@
 Text Notes 23250 13650 0    100  ~ 0
 To bypass inverting opamp populate:\nR13 and R16 with 1K resistors, R22 0R,\nomit others
+Text Notes 18050 16250 0    100  ~ 0
+Expect increasing negative voltage on TP10 and TP12 as U4A output voltage increases. \nTP9 should remain at GND (some offset normal).\nThe output is inverted by U4B so TP14 should increase inversely proportional to TP10 and TP12.
+Text Notes 17400 9500 0    100  ~ 0
+Expect increasing positive voltage on TP8 and TP11 as U3A output voltage increases. \nTP7 should remain at GND (some offset normal).
 $EndSCHEMATC

Commit message: updates
Other:
- note added: "N-Channel\nPower Mosfet\nIPP80N03S4L03AKSA1\nhttps://www.mouser.com/ds/2/196/Infineon-IPB80N03S4L_03_IPP_I80N03S4L_04-DS-v02_01-1226077.pdf"
- note added: "P-Channel\nPower Mosfet\n IPP80P03P4L-04\nhttps://www.infineon.com/dgdl/Infineon-I80P03P4L_04-DS-v01_01-en.pdf?fileId=db3a30431ddc9372011e07e95eb827d7"
- note removed: "N-Channel\nPower Mosfet"
- note removed: "P-Channel\nPower Mosfet"
Changed lines of the file:
@@
 Text Label 28900 8650 2    50   ~ 0
 DUT_POS
-Text Notes 14650 5050 0    50   ~ 0
-N-Channel\nPower Mosfet
+Text Notes 14725 5150 0    50   ~ 0
+N-Channel\nPower Mosfet\nIPP80N03S4L03AKSA1\nhttps://www.mouser.com/ds/2/196/Infineon-IPB80N03S4L_03_IPP_I80N03S4L_04-DS-v02_01-1226077.pdf
 Text Notes 13675 7225 0    50   ~ 0
 Power Resistor\nArcol HS100 \n1ohm 100W
-Text Notes 14750 15650 0    50   ~ 0
-P-Channel\nPower Mosfet
+Text Notes 14550 15625 0    50   ~ 0
+P-Channel\nPower Mosfet\n IPP80P03P4L-04\nhttps://www.infineon.com/dgdl/Infineon-I80P03P4L_04-DS-v01_01-en.pdf?fileId=db3a30431ddc9372011e07e95eb827d7
 Text Notes 19700 6750 0    50   ~ 0
 InstGain: 14dB
