File: HW/CurrentSinkModule/CurrentSinkModule/CurrentSink.sch (KiCad schematic (older format))
At the start: 101 parts, among them J1 Conn_01x03, J2 Conn_01x03, J3 MosfetSocketx3, J4 MosfetSocketx3, U1 LTC2058, U2 LTC2058, U3 LTC2058, U4 LTC2058

Commit message: updated
Other:
- note added: "N-Channel\nPower Mosfet\nIXFK50N85X\nhttps://www.littelfuse.com/~/media/electronics/datasheets/discrete_mosfets/littelfuse_discrete_mosfets_n-channel_ultra_junction_ixf_50n85x_datasheet.pdf.pdf"
- note added: "P-Channel\nPower Mosfet\nIXTK90P20P\nhttps://m.littelfuse.com/~/media/electronics/datasheets/discrete_mosfets/littelfuse_discrete_mosfets_p-channel_ixt_90p20p_datasheet.pdf.pdf"
- note removed: "N-Channel\nPower Mosfet\nIPP80N03S4L03AKSA1\nhttps://www.mouser.com/ds/2/196/Infineon-IPB80N03S4L_03_IPP_I80N03S4L_04-DS-v02_01-1226077.pdf"
- note removed: "P-Channel\nPower Mosfet\n IPP80P03P4L-04\nhttps://www.infineon.com/dgdl/Infineon-I80P03P4L_04-DS-v01_01-en.pdf?fileId=db3a30431ddc9372011e07e95eb827d7"
Changed lines of the file:
@@
 Text Label 28900 8650 2    50   ~ 0
 DUT_POS
-Text Notes 14725 5150 0    50   ~ 0
-N-Channel\nPower Mosfet\nIPP80N03S4L03AKSA1\nhttps://www.mouser.com/ds/2/196/Infineon-IPB80N03S4L_03_IPP_I80N03S4L_04-DS-v02_01-1226077.pdf
+Text Notes 14575 4325 0    50   ~ 0
+N-Channel\nPower Mosfet\nIXFK50N85X\nhttps://www.littelfuse.com/~/media/electronics/datasheets/discrete_mosfets/littelfuse_discrete_mosfets_n-channel_ultra_junction_ixf_50n85x_datasheet.pdf.pdf
 Text Notes 13675 7225 0    50   ~ 0
 Power Resistor\nArcol HS100 \n1ohm 100W
 Text Notes 14550 15625 0    50   ~ 0
-P-Channel\nPower Mosfet\n IPP80P03P4L-04\nhttps://www.infineon.com/dgdl/Infineon-I80P03P4L_04-DS-v01_01-en.pdf?fileId=db3a30431ddc9372011e07e95eb827d7
+P-Channel\nPower Mosfet\nIXTK90P20P\nhttps://m.littelfuse.com/~/media/electronics/datasheets/discrete_mosfets/littelfuse_discrete_mosfets_p-channel_ixt_90p20p_datasheet.pdf.pdf
 Text Notes 19700 6750 0    50   ~ 0
 InstGain: 14dB

Commit message: updated
Parts:
- added R29, R30: 1M, symbol Device:R
Connections:
- net DACSIG1: now also R29.1
- net DACSIG2: now also R30.1
- net GNDS: now also R29.2, R30.2
Other:
- note added: "DRAIN\nGATE\nSOURCE"
Changed lines of the file:
@@
 Wire Wire Line
 	1900 20600 1950 20600
-Text Label 2575 15200 0    50   ~ 0
+Text Label 1325 15200 0    50   ~ 0
 DACSIG2
-Text Label 2575 6300 0    50   ~ 0
+Text Label 1325 6300 0    50   ~ 0
 DACSIG1
 $Comp
@@
 	3750 6300 3950 6300
 Wire Wire Line
-	2575 6300 3200 6300
+	1325 6300 2425 6300
 $Comp
 L Device:C C4
@@
 	3750 15200 3950 15200
 Wire Wire Line
-	2575 15200 3200 15200
+	1325 15200 2425 15200
 $Comp
 L Device:C C3
@@
 Wire Wire Line
 	4850 16400 4850 16275
+$Comp
+L Device:R R30
+U 1 1 5DE88293
+P 2425 15850
+F 0 "R30" H 2495 15895 50  0000 L CNN
+F 1 "1M" H 2495 15806 50  0000 L CNN
+F 2 "" V 2355 15850 50  0001 C CNN
+F 3 "~" H 2425 15850 50  0001 C CNN
+	1    2425 15850
+	1    0    0    -1
+$EndComp
+Wire Wire Line
+	2425 15700 2425 15200
+Connection ~ 2425 15200
+Wire Wire Line
+	2425 15200 3200 15200
+Wire Wire Line
+	2425 16000 2425 16400
+Wire Wire Line
+	2425 16400 3200 16400
+Connection ~ 3200 16400
+$Comp
+L Device:R R29
+U 1 1 5DECD66E
+P 2425 6950
+F 0 "R29" H 2495 6995 50  0000 L CNN
+F 1 "1M" H 2495 6906 50  0000 L CNN
+F 2 "" V 2355 6950 50  0001 C CNN
+F 3 "~" H 2425 6950 50  0001 C CNN
+	1    2425 6950
+	1    0    0    -1
+$EndComp
+Wire Wire Line
+	2425 6800 2425 6300
+Wire Wire Line
+	2425 7100 2425 7500
+Wire Wire Line
+	2425 7500 3200 7500
+Connection ~ 2425 6300
+Wire Wire Line
+	2425 6300 3200 6300
+Text Notes 14000 4750 0    50   ~ 0
+DRAIN\nGATE\nSOURCE
+Text Notes 13975 16025 0    50   ~ 0
+DRAIN\nGATE\nSOURCE
 $EndSCHEMATC
