File: HW/CurrentSinkModule/CurrentSinkModule/CurrentSinkModule.kicad_pcb (KiCad board)
At the start: 4 copper layers, 108.6 x 114.3 mm, 35 parts, among them U3 LTC2058, U4 LTC2058

Commit message: updated
Parts:
- removed Q_NEGMOS1: IRF5210, Package_TO_SOT_THT:TO-220-3_Vertical
- removed Q_POSMOS1: IRF3710, Package_TO_SOT_THT:TO-220-3_Vertical
- added C1: C, Capacitor_SMD:C_0402_1005Metric, F.Cu at (250.1, -8.00)
- added C10: 4.7u, Capacitor_SMD:C_0402_1005Metric, F.Cu at (258.8, -28.1)
- added C11: 10n, Capacitor_SMD:C_0402_1005Metric, F.Cu at (247.7, -3.95)
- added C12: 10n, Capacitor_SMD:C_0402_1005Metric, F.Cu at (253.3, -9.99)
- added C13: 1n 5% Mica/C0G, Capacitor_SMD:C_0402_1005Metric, F.Cu at (244.8, -1.96)
- added C14: 1n 5% Mica/C0G, Capacitor_SMD:C_0402_1005Metric, F.Cu at (248.9, -5.94)
- added C15: 1n 5% Mica/C0G, Capacitor_SMD:C_0402_1005Metric, F.Cu at (239.0, -1.48)
- added C16: 1n 5% Mica/C0G, Capacitor_SMD:C_0402_1005Metric, F.Cu at (244.2, -7.93)
- added C17: 22n, Capacitor_SMD:C_0402_1005Metric, F.Cu at (246.0, -16.0)
- added C18: 22n, Capacitor_SMD:C_0402_1005Metric, F.Cu at (251.8, -22.1)
- added C19: 330n, Capacitor_SMD:C_0402_1005Metric, F.Cu at (251.8, -24.1)
- added C2: C, Capacitor_SMD:C_0402_1005Metric, F.Cu at (257.6, -16.1)
- added C20: 330n, Capacitor_SMD:C_0402_1005Metric, F.Cu at (224.0, -1.46)
- added C21: 330n, Capacitor_SMD:C_0402_1005Metric, F.Cu at (215.3, -2.16)
- added C22: 330n, Capacitor_SMD:C_0402_1005Metric, F.Cu at (218.2, -1.46)
- added C23: 10n, Capacitor_SMD:C_0402_1005Metric, F.Cu at (233.2, -2.61)
- added C24: 10n, Capacitor_SMD:C_0402_1005Metric, F.Cu at (253.3, -12.0)
- added C25: 10n, Capacitor_SMD:C_0402_1005Metric, F.Cu at (254.7, -14.1)
- added C26: 10n, Capacitor_SMD:C_0402_1005Metric, F.Cu at (244.8, -3.95)
- added C27: 4.7u, Capacitor_SMD:C_0402_1005Metric, F.Cu at (250.4, -9.99)
- added C28: 4.7u, Capacitor_SMD:C_0402_1005Metric, F.Cu at (241.9, -1.48)
- added C29: 10n, Capacitor_SMD:C_0402_1005Metric, F.Cu at (246.0, -5.94)
- added C3: C, Capacitor_SMD:C_0402_1005Metric, F.Cu at (251.8, -14.0)
- added C30: 10n, Capacitor_SMD:C_0402_1005Metric, F.Cu at (257.7, -18.1)
- added C31: 4.7u, Capacitor_SMD:C_0402_1005Metric, F.Cu at (247.2, -7.93)
- added C32: 4.7u, Capacitor_SMD:C_0402_1005Metric, F.Cu at (254.7, -16.1)
- added C33: 10n, Capacitor_SMD:C_0402_1005Metric, F.Cu at (250.4, -12.0)
- added C34: 10n, Capacitor_SMD:C_0402_1005Metric, F.Cu at (237.3, -5.46)
- added C4: C, Capacitor_SMD:C_0402_1005Metric, F.Cu at (241.9, -3.47)
- added C5: 4.7u, Capacitor_SMD:C_0402_1005Metric, F.Cu at (221.1, -1.46)
- added C6: 4.7u, Capacitor_SMD:C_0402_1005Metric, F.Cu at (225.4, -21.7)
- added C7: 10n, Capacitor_SMD:C_0402_1005Metric, F.Cu at (210.6, -1.31)
- added C8: 10n, Capacitor_SMD:C_0402_1005Metric, F.Cu at (215.3, -8.06)
- added C9: 4.7u, Capacitor_SMD:C_0402_1005Metric, F.Cu at (241.6, -11.9)
- added D1: D_Schottky, Diode_SMD:D_SOD-123, F.Cu at (267.4, -20.7)
- added D2: D_Schottky, Diode_SMD:D_SOD-123, F.Cu at (273.1, -27.4)
- added D3: 3V3, Diode_SMD:D_SOD-123, F.Cu at (216.7, -4.83)
- added D4: 3V3, Diode_SMD:D_SOD-123, F.Cu at (230.6, -21.0)
- added D5: D_Schottky, Diode_SMD:D_SOD-123, F.Cu at (267.4, -24.1)
- added D6: D_Schottky, Diode_SMD:D_SOD-123, F.Cu at (267.4, -27.4)
- added GND1: TestPoint, TestPoint:TestPoint_Pad_2.0x2.0mm, F.Cu at (229.7, -2.08)
- added GND10: TestPoint, TestPoint:TestPoint_Pad_2.0x2.0mm, F.Cu at (238.2, -12.5)
- added GND11: TestPoint, TestPoint:TestPoint_Pad_2.0x2.0mm, F.Cu at (233.8, -9.68)
- added GND12: TestPoint, TestPoint:TestPoint_Pad_2.0x2.0mm, F.Cu at (282.1, -27.1)
- added GND2: TestPoint, TestPoint:TestPoint_Pad_2.0x2.0mm, F.Cu at (233.8, -5.63)
- added GND3: TestPoint, TestPoint:TestPoint_Pad_2.0x2.0mm, F.Cu at (255.3, -27.1)
- added GND4: TestPoint, TestPoint:TestPoint_Pad_2.0x2.0mm, F.Cu at (237.9, -8.48)
- added GND5: TestPoint, TestPoint:TestPoint_Pad_2.0x2.0mm, F.Cu at (248.4, -19.0)
- added GND6: TestPoint, TestPoint:TestPoint_Pad_2.0x2.0mm, F.Cu at (242.5, -14.9)
- added GND7: TestPoint, TestPoint:TestPoint_Pad_2.0x2.0mm, F.Cu at (244.3, -19.0)
- added GND8: TestPoint, TestPoint:TestPoint_Pad_2.0x2.0mm, F.Cu at (248.4, -23.0)
- added GND9: TestPoint, TestPoint:TestPoint_Pad_2.0x2.0mm, F.Cu at (280.4, -23.0)
- added J1: Conn_01x03, Connector_PinHeader_2.54mm:PinHeader_1x03_P2.54mm_Vertical, F.Cu at (211.5, -9.68)
- added J2: Conn_01x03, Connector_PinHeader_2.54mm:PinHeader_1x03_P2.54mm_Vertical, F.Cu at (221.6, -26.8)
- added J3: MosfetSocketx3, TerminalBlock:TerminalBlock_bornier-3_P5.08mm, F.Cu at (198.0, 73.3)
- added J4: MosfetSocketx3, TerminalBlock:TerminalBlock_bornier-3_P5.08mm, F.Cu at (187.8, 141.9)
- added JP5: BYPASS, Jumper:SolderJumper-2_P1.3mm_Open_Pad1.0x1.5mm, F.Cu at (234.3, -17.5)
- added JP6: BYPASS, Jumper:SolderJumper-2_P1.3mm_Open_Pad1.0x1.5mm, F.Cu at (229.9, -17.5)
- added JP7: BYPASS, Jumper:SolderJumper-2_P1.3mm_Open_Pad1.0x1.5mm, F.Cu at (229.9, -14.0)
- added JP8: BYPASS, Jumper:SolderJumper-2_P1.3mm_Open_Pad1.0x1.5mm, F.Cu at (243.0, -27.3)
- added R1: R, Resistor_SMD:R_0402_1005Metric, F.Cu at (241.6, -9.92)
- added R10: 22K 1%, Resistor_SMD:R_0402_1005Metric, F.Cu at (257.7, -24.1)
- added R11: 22K 1%, Resistor_SMD:R_0402_1005Metric, F.Cu at (251.8, -18.1)
- added R12: 22K 1%, Resistor_SMD:R_0402_1005Metric, F.Cu at (241.3, -7.93)
- added R13: 100R, Resistor_SMD:R_0402_1005Metric, F.Cu at (240.2, -5.46)
- added R14: 0R, Resistor_SMD:R_0402_1005Metric, F.Cu at (244.5, -9.92)
- added R15: 0R, Resistor_SMD:R_0402_1005Metric, F.Cu at (254.7, -20.1)
- added R16: 100R, Resistor_SMD:R_0402_1005Metric, F.Cu at (257.7, -22.1)
- added R17: R, Resistor_SMD:R_0402_1005Metric, F.Cu at (248.9, -14.0)
- added R18: R, Resistor_SMD:R_0402_1005Metric, F.Cu at (247.5, -12.0)
- added R19: R, Resistor_SMD:R_0402_1005Metric, F.Cu at (251.8, -16.0)
- added R2: R, Resistor_SMD:R_0402_1005Metric, F.Cu at (251.8, -20.1)
- added R20: R, Resistor_SMD:R_0402_1005Metric, F.Cu at (239.0, -3.47)
- added R21: R, Resistor_SMD:R_0805_2012Metric_Pad1.15x1.40mm_HandSolder, F.Cu at (235.9, -21.2)
- added R22: R, Resistor_SMD:R_0402_1005Metric, F.Cu at (254.7, -18.1)
- added R23: 0R, Resistor_SMD:R_0402_1005Metric, F.Cu at (243.1, -5.94)
- added R24: R, Resistor_SMD:R_0805_2012Metric_Pad1.15x1.40mm_HandSolder, F.Cu at (216.2, -10.5)
- added R25: R, Resistor_SMD:R_0402_1005Metric, F.Cu at (247.5, -9.99)
- added R26: R, Resistor_SMD:R_0402_1005Metric, F.Cu at (257.7, -20.1)
- added R3: R, Resistor_SMD:R_0402_1005Metric, F.Cu at (254.7, -24.1)
- added R4: R, Resistor_SMD:R_0402_1005Metric, F.Cu at (254.7, -22.1)
- added R5: R, Resistor_SMD:R_0402_1005Metric, F.Cu at (258.8, -26.1)
- added R6: R, Resistor_SMD:R_0402_1005Metric, F.Cu at (244.5, -11.9)
- added R7: R, Resistor_SMD:R_0402_1005Metric, F.Cu at (246.0, -14.0)
- added R8: R, Resistor_SMD:R_0402_1005Metric, F.Cu at (248.9, -16.0)
- added R9: 22K 1%, Resistor_SMD:R_0402_1005Metric, F.Cu at (236.1, -2.61)
- added TP1: TestPoint, TestPoint:TestPoint_Pad_2.0x2.0mm, F.Cu at (276.3, -23.0)
- added TP10: TestPoint, TestPoint:TestPoint_Pad_2.0x2.0mm, F.Cu at (234.1, -13.7)
- added TP11: TestPoint, TestPoint:TestPoint_Pad_2.0x2.0mm, F.Cu at (247.2, -27.1)
- added TP12: TestPoint, TestPoint:TestPoint_Pad_2.0x2.0mm, F.Cu at (229.8, -10.2)
- added TP13: TestPoint, TestPoint:TestPoint_Pad_2.0x2.0mm, F.Cu at (240.3, -20.6)
- added TP14: TestPoint, TestPoint:TestPoint_Pad_2.0x2.0mm, F.Cu at (221.6, -4.48)
- added TP15: TestPoint, TestPoint:TestPoint_Pad_2.0x2.0mm, F.Cu at (278.0, -27.1)
- added TP16: TestPoint, TestPoint:TestPoint_Pad_2.0x2.0mm, F.Cu at (272.3, -23.7)
- added TP2: TestPoint, TestPoint:TestPoint_Pad_2.0x2.0mm, F.Cu at (272.3, -19.7)
- added TP3: TestPoint, TestPoint:TestPoint_Pad_2.0x2.0mm, F.Cu at (251.3, -27.1)
- added TP4: TestPoint, TestPoint:TestPoint_Pad_2.0x2.0mm, F.Cu at (244.3, -23.0)
- added TP7: TestPoint, TestPoint:TestPoint_Pad_2.0x2.0mm, F.Cu at (229.8, -6.13)
- added TP8: TestPoint, TestPoint:TestPoint_Pad_2.0x2.0mm, F.Cu at (238.5, -16.6)
- added TP9: TestPoint, TestPoint:TestPoint_Pad_2.0x2.0mm, F.Cu at (225.6, -4.48)
- added U1: LTC2058, Package_SO:SOIC-8_3.9x4.9mm_P1.27mm, F.Cu at (236.6, -25.9)
- added U2: LTC2058, Package_SO:SOIC-8_3.9x4.9mm_P1.27mm, F.Cu at (223.5, -9.73)
- added U_NEGIA1: INA128UA, Package_SO:SOIC-8_3.9x4.9mm_P1.27mm, F.Cu at (223.5, -16.2)
- added U_POSIA1: INA128UA, Package_SO:SOIC-8_3.9x4.9mm_P1.27mm, F.Cu at (228.2, -25.9)
- turned J_SUTPOS1 to 180 degrees
Routing:
- net Net-(J3-Pad3): track 30.2 -> 17.4 mm
- net Net-(J4-Pad1): track 55.4 -> 46.0 mm
- net Net-(J4-Pad3): track 47.3 -> 52.4 mm
- net /CurrentSink/DUT_POS: track 29.2 -> 25.2 mm
- net Net-(J3-Pad1): track 32.7 -> 28.9 mm
- net /CurrentSink/DUT_NEG: track 26.3 -> 27.4 mm

Commit message: Updates
- New simplified current sink design: see LTSpice model "MOSFET_CurrentSense_NoSignalInversion".
Needs to be confirmed on breadboard!
Parts:
- C10, C11, C12, C19, C20, C21, C22, C23, C24, C25, C26, C27, C28, C29, C30, C31, C32, C33, C34, C5, C6, C7, C8, C9, JP5, JP7: moved to B.Cu
- moved R3 275.7 mm to (129.7, 221.6), turned to 180 degrees
- moved R5 275.0 mm to (142.0, 222.9), turned to 180 degrees
- moved TP3 270.6 mm to (129.8, 214.8)
- moved U1 267.9 mm to (135.6, 222.2)
- moved R19 265.3 mm to (129.7, 219.6), turned to 180 degrees
- moved R17 265.2 mm to (129.7, 222.9)
- moved C6 264.6 mm to (133.1, 226.3)
- moved R8 262.8 mm to (142.0, 224.2)
- moved C3 262.4 mm to (129.7, 218.3), turned to 180 degrees
- moved C1 261.6 mm to (129.7, 224.3)
- moved JP5 259.1 mm to (133.1, 221.0), turned to 90 degrees
- moved GND8 259.1 mm to (290.7, 232.5)
- moved R7 257.5 mm to (142.0, 221.6), turned to 180 degrees
- moved JP7 254.6 mm to (138.3, 223.5), turned to 90 degrees
- moved R1 253.1 mm to (129.7, 217.0)
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Routing:
- net Net-(C3-Pad1): track 0.00 -> 17.9 mm, vias 0 -> 2
- net -5VA: track 0.00 -> 15.5 mm, vias 0 -> 3
- net +5VA: track 0.00 -> 15.2 mm, vias 0 -> 3
- net -5V: track 0.00 -> 13.9 mm, vias 0 -> 3
- net +5V: track 0.00 -> 13.0 mm, vias 0 -> 3
- net Net-(JP7-Pad2): track 0.00 -> 7.27 mm, vias 0 -> 1
- net Net-(JP5-Pad1): track 0.00 -> 7.23 mm, vias 0 -> 1
- net Net-(C3-Pad2): track 0.00 -> 5.77 mm
- net Net-(R19-Pad2): track 0.00 -> 5.35 mm
- net Net-(R5-Pad2): track 0.00 -> 3.39 mm
- net /CurrentSink/DACSIG2: track 0.00 -> 2.69 mm
- net Net-(J1-Pad1): track 0.00 -> 2.54 mm
- net Net-(C1-Pad1): track 0.00 -> 1.40 mm
- net GNDS: track 0.00 -> 0.78 mm, vias 0 -> 1
- removed copper zone on In1.Cu, net +12V
- removed copper zone on In2.Cu, net -12V
Other:
- outline, holes or cut-outs redrawn
- copper layers 4 -> 2

Commit message: Finished CurrentSinkRevC layout
Parts:
- removed D5, D6: D_Schottky, Diode_SMD:D_SOD-123
- removed GND12, TP15, TP16: TestPoint, TestPoint:TestPoint_Pad_2.0x2.0mm
- removed JPWR2: Conn_01x03, Connector_Molex:Molex_KK-254_AE-6410-03A_1x03_P2.54mm_Vertical
- removed the REF** at (271.7, 160.0)
- removed the REF** at (141.4, 35.7)
- removed the REF** at (271.7, 55.9)
- added REF**: MountingHole_4.3mm_M4_ISO14580, MountingHole:MountingHole_4.3mm_M4_ISO14580, F.Cu at (273.5, 120.4)
- added REF**: MountingHole_4.3mm_M4_ISO14580, MountingHole:MountingHole_4.3mm_M4_ISO14580, F.Cu at (273.6, 152.9)
- added REF**: MountingHole_4.3mm_M4_ISO14580, MountingHole:MountingHole_4.3mm_M4_ISO14580, F.Cu at (273.3, 64.3)
- JP1, JP2, JP3, JP4: footprint Jumper:SolderJumper-2_P1.3mm_Bridged_Pad1.0x1.5mm -> Jumper:SolderJumper-2_P1.3mm_Open_Pad1.0x1.5mm
- JP7: moved to F.Cu
- moved GND2 133.0 mm to (243.2, 151.5)
- moved C4 132.0 mm to (246.3, 64.1), turned to 180 degrees
- moved C2 131.4 mm to (246.3, 69.3)
- moved R20 129.6 mm to (246.3, 65.5), turned to 180 degrees
- moved GND1 128.5 mm to (239.8, 68.0)
- moved TP3 126.7 mm to (239.6, 151.5)
- moved R4 126.5 mm to (246.3, 68.0), turned to 180 degrees
- moved R18 125.8 mm to (246.3, 70.6)
- moved JP6 125.5 mm to (252.1, 62.1), turned to 180 degrees
- moved JP7 125.5 mm to (235.5, 144.1), turned to 0 degrees
- moved R2 124.9 mm to (245.4, 62.8), turned to 180 degrees
- moved R8 124.4 mm to (234.1, 140.5)
- moved GND7 123.6 mm to (236.6, 84.4)
- moved C5 123.6 mm to (230.3, 137.9)
- moved C7 123.6 mm to (230.3, 136.0)
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Connections:
- C10 pad 1: -5V -> -12V
- C11 pad 1: +5V -> +12V
- C12 pad 1: -5V -> -12V
- C19 pad 2: +5V -> +12V
- C20 pad 2: -5V -> -12V
- C21 pad 2: +5VA -> +12V
- C22 pad 2: -5VA -> -12V
- C23 pad 1: +5V -> +12V
- C24 pad 1: -5V -> -12V
- C25 pad 1: +5VA -> +12V
- C26 pad 1: -5VA -> -12V
- C27 pad 1: +5V -> +12V
- C28 pad 1: -5V -> -12V
- C29 pad 1: +5V -> +12V
- C30 pad 1: -5V -> -12V
- C31 pad 1: +5VA -> +12V
- C32 pad 1: -5VA -> -12V
- C33 pad 1: +5VA -> +12V
- C34 pad 1: -5VA -> -12V
- C5 pad 1: +5VA -> +12V
- C6 pad 1: -5VA -> -12V
- C7 pad 1: +5VA -> +12V
- C8 pad 1: -5VA -> -12V
- C9 pad 1: +5V -> +12V
- D1 pad 1: +5V -> +12V
- D2 pad 2: -5V -> -12V
- JP7 pad 1: Net-(C3-Pad1) -> Net-(JP7-Pad1)
- JP7 pad 2: Net-(JP7-Pad2) -> Net-(J1-Pad1)
- JP8 pad 1: Net-(C4-Pad1) -> Net-(JP8-Pad1)
- R25 pad 1: Net-(R25-Pad1) -> Net-(C4-Pad1)
- R25 pad 2: Net-(J2-Pad1) -> Net-(R25-Pad2)
- R26 pad 2: Net-(R25-Pad1) -> Net-(R25-Pad2)
- R5 pad 1: Net-(J1-Pad1) -> GNDS
- R6 pad 1: Net-(R25-Pad1) -> Net-(J2-Pad1)
- R6 pad 2: Net-(R6-Pad2) -> Net-(JP8-Pad1)
- R7 pad 1: Net-(J1-Pad1) -> Net-(C3-Pad1)
- R7 pad 2: Net-(JP7-Pad2) -> Net-(JP7-Pad1)
- R8 pad 1: GNDS -> Net-(JP7-Pad1)
- TP1 pad 1: -5V -> -12V
- TP2 pad 1: +5V -> +12V
- U1 pad 4: -5VA -> -12V
- U1 pad 5: Net-(C3-Pad1) -> Net-(R5-Pad2)
- U1 pad 6: Net-(R5-Pad2) -> Net-(JP7-Pad1)
- U1 pad 7: Net-(JP7-Pad2) -> Net-(J1-Pad1)
- U1 pad 8: +5VA -> +12V
- U2 pad 4: -5V -> -12V
- U2 pad 5: Net-(C4-Pad1) -> Net-(R25-Pad2)
- U2 pad 6: Net-(R6-Pad2) -> Net-(JP8-Pad1)
- U2 pad 8: +5V -> +12V
- U3 pad 4: -5V -> -12V
- U3 pad 8: +5V -> +12V
- U4 pad 1: /CurrentSink/ADCSIG2 -> Net-(J4-Pad1)
- U4 pad 2: Net-(R13-Pad1) -> Net-(R21-Pad2)
- U4 pad 3: Net-(R22-Pad1) -> Net-(J1-Pad2)
- U4 pad 4: -5VA -> -12V
- U4 pad 5: Net-(R21-Pad2) -> Net-(R22-Pad1)
- U4 pad 6: Net-(J1-Pad2) -> Net-(R13-Pad1)
- U4 pad 7: Net-(J4-Pad1) -> /CurrentSink/ADCSIG2
- U4 pad 8: +5VA -> +12V
- U_NEGIA1 pad 4: -5VA -> -12V
- U_NEGIA1 pad 7: +5VA -> +12V
- U_POSIA1 pad 4: -5V -> -12V
- U_POSIA1 pad 7: +5V -> +12V
Routing:
- net Net-(J3-Pad3): track 17.4 -> 134.6 mm
- net Net-(J3-Pad1): track 28.9 -> 98.4 mm
- net Net-(R14-Pad2): track 0.00 -> 56.9 mm
- net GNDS: track 0.78 -> 51.4 mm, vias 1 -> 25
- net /CurrentSink/ADCSIG1: track 0.00 -> 46.1 mm
- net Net-(R13-Pad2): track 0.00 -> 43.8 mm
- net Net-(J4-Pad3): track 52.4 -> 95.9 mm
- net -12V: track 0.00 -> 36.2 mm, vias 0 -> 7
- net +12V: track 0.00 -> 36.0 mm, vias 0 -> 7
- net Net-(J4-Pad1): track 46.0 -> 77.8 mm
- net /CurrentSink/ADCSIG2: track 0.00 -> 27.8 mm
- net Net-(J2-Pad1): track 0.00 -> 27.5 mm
- net Net-(J1-Pad1): track 2.54 -> 28.5 mm
- net Net-(C13-Pad1): track 0.00 -> 25.4 mm
- net Net-(C15-Pad1): track 0.00 -> 24.0 mm
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- added copper zone on F.Cu, net (none)
- added copper zone on In1.Cu, net +12V
- added copper zone on In2.Cu, net -12V
Other:
- board size 108.6 x 114.3 mm -> 100.3 x 100.3 mm
- copper layers 2 -> 4
- board text added: "+12V"
- board text added: "-12V"
- board text added: "CurrentSink RevC C.Sutton © 2919"
- board text removed: "CurrentModule RevC C.Sutton © 1919"

Commit message: Added Interafec IBOMS
Parts:
- removed the REF** at (-88.1, 126.8)
- added JP10: BYPASS, Jumper:SolderJumper-2_P1.3mm_Open_Pad1.0x1.5mm, F.Cu at (260.7, 89.5)
- added JP9: BYPASS, Jumper:SolderJumper-2_P1.3mm_Open_Pad1.0x1.5mm, F.Cu at (259.7, 133.6)
- JP5: moved to F.Cu
- moved JP5 17.3 mm to (241.4, 145.4)
- moved R7 9.57 mm to (225.3, 135.4), turned to 90 degrees
- moved R8 6.39 mm to (230.1, 135.4), turned to 270 degrees
- moved JP7 4.32 mm to (235.3, 139.8), turned to 90 degrees
- moved GND2 3.41 mm to (241.3, 154.3), turned to 90 degrees
- moved TP3 3.10 mm to (238.3, 154.3)
- moved R5 1.21 mm to (234.1, 142.9)
- moved GND4 0.09 mm to (251.7, 133.6), turned to 180 degrees
Routing:
- net Net-(JP5-Pad1): track 8.79 -> 26.8 mm, vias 1 -> 0
- net Net-(J1-Pad1): track 28.5 -> 18.8 mm
- net Net-(C3-Pad1): track 21.7 -> 29.5 mm, vias 1 -> 0
- net /CurrentSink/ADCSIG2: track 27.8 -> 31.1 mm
- net Net-(JP9-Pad1): track 43.8 -> 45.9 mm
- net Net-(JP7-Pad1): track 15.4 -> 17.4 mm
- net Net-(R5-Pad2): track 3.39 -> 4.60 mm
- net /CurrentSink/DACSIG2: track 24.8 -> 24.0 mm
Other:
- board text added: "BYPASS IN FILTER"
- board text added: "BYPASS INPUT"
- board text added: "BYPASS OUTPUT"

Commit message: current module hw update
- Deleted opamp Bypass jumpers in schematic; they break opamp configurations
- Added bypass instructions in schematic for each opamp.
Changed lines of the file:
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@@
-(kicad_pcb (version 20171130) (host pcbnew "(5.1.2-1)-1")
+(kicad_pcb (version 20171130) (host pcbnew "(5.1.2)-2")
   (general
     (thickness 1.6)
@@
     (tags resistor)
     (attr smd)
-    (fp_text reference R8 (at 2.9845 0 90) (layer F.SilkS)
+    (fp_text reference R8 (at -1.8669 0.0254 180) (layer F.SilkS)
       (effects (font (size 0.8 0.8) (thickness 0.15)))
     )
@@
     (tags resistor)
     (attr smd)
-    (fp_text reference R7 (at -2.9845 0 90) (layer F.SilkS)
-      (effects (font (size 0.8 0.8) (thickness 0.15)))
-    )
+    (fp_text reference R7 (at 1.9304 0 180) (layer F.SilkS)
+      (effects (font (size 0.8 0.8) (thickness 0.15)))
+    )

Commit message: Tested RevC LTC3260 fixes
- updated passive LTC3260 component values
Parts:
- added REF**: 1458G4, 1458G4_OUTLINE:1458G4, F.Cu at (214.8, 133.0)
Changed lines of the file:
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@@
     (tracks 461)
     (zones 0)
-    (modules 132)
+    (modules 133)
     (nets 50)
   )
@@
     (add_net "Net-(R5-Pad2)")
   )
+  (module 1458G4_OUTLINE:1458G4 locked (layer F.Cu)
+    (at 214.757 132.969)
+    (fp_text reference REF** (at -80.01 -96.52) (layer F.SilkS) hide
+      (effects (font (size 1 1) (thickness 0.15)))
+    )
+    (fp_text value 1458G4 (at -80.01 -93.98) (layer F.Fab)
+      (effects (font (size 1 1) (thickness 0.15)))
+    )
+    (fp_line (start -125.73 87.63) (end -125.73 -86.36) (layer Dwgs.User) (width 0.15))
+    (fp_line (start 124.46 87.63) (end -125.73 87.63) (layer Dwgs.User) (width 0.15))
+    (fp_line (start 124.46 -86.36) (end 124.46 87.63) (layer Dwgs.User) (width 0.15))
+    (fp_line (start -125.73 -86.36) (end 124.46 -86.36) (layer Dwgs.User) (width 0.15))
+    (fp_line (start 73.66 -86.36) (end 73.66 87.63) (layer F.SilkS) (width 0.15))
+    (fp_line (start 73.66 -55.88) (end 124.46 -55.88) (layer F.SilkS) (width 0.15))
+    (fp_line (start -125.73 36.83) (end 73.66 36.83) (layer F.SilkS) (width 0.15))
+    (fp_line (start 73.66 57.15) (end 124.46 57.15) (layer F.SilkS) (width 0.15))
+    (fp_text user "IEC Input" (at 99.06 -81.28) (layer F.SilkS)
+      (effects (font (size 2 2) (thickness 0.15)))
+    )
+    (fp_text user "Analog Section" (at 56.388 -81.28) (layer F.SilkS)
+      (effects (font (size 2 2) (thickness 0.15)))
+    )
+    (fp_text user "Front Panel" (at 58.42 81.28) (layer F.SilkS)
+      (effects (font (size 2 2) (thickness 0.15)))
+    )
+    (fp_text user "Front Connectors" (at 99.06 81.28) (layer F.SilkS)
+      (effects (font (size 2 2) (thickness 0.15)))
+    )
+    (fp_text user "Power Supply" (at 100.33 2.54) (layer F.SilkS)
+      (effects (font (size 2 2) (thickness 0.15)))
+    )
+  )
   (module FischerElectronikFanHeatsink:LAM_5_100_12 locked (layer F.Cu)
