File: HW/IsolatedThreeOutputSMPS/ExternRegulatedConverters/18VIN_ExternRegulatedConverter_12D_12S_5S/PowerFlags.sch (KiCad schematic (older format))
At the start: 0 parts

Commit message: RevA layout PSU
Changed lines of the file:
@@
 	-1   0    0    1
 $EndComp
-$Comp
-L power:PWR_FLAG #FLG01
-U 1 1 5D491B70
-P 3550 3375
-F 0 "#FLG01" H 3550 3450 50  0001 C CNN
-F 1 "PWR_FLAG" H 3550 3546 50  0000 C CNN
-F 2 "" H 3550 3375 50  0001 C CNN
-F 3 "~" H 3550 3375 50  0001 C CNN
-	1    3550 3375
-	-1   0    0    1
-$EndComp
-$Comp
-L power:PWR_FLAG #FLG03
-U 1 1 5D49173E
-P 4925 3975
-F 0 "#FLG03" H 4925 4050 50  0001 C CNN
-F 1 "PWR_FLAG" H 4925 4146 50  0000 C CNN
-F 2 "" H 4925 3975 50  0001 C CNN
-F 3 "~" H 4925 3975 50  0001 C CNN
-	1    4925 3975
-	1    0    0    -1
-$EndComp
-$Comp
-L power:PWR_FLAG #FLG02
-U 1 1 5D49135F
-P 4925 3375
-F 0 "#FLG02" H 4925 3450 50  0001 C CNN
-F 1 "PWR_FLAG" H 4925 3546 50  0000 C CNN
-F 2 "" H 4925 3375 50  0001 C CNN
-F 3 "~" H 4925 3375 50  0001 C CNN
-	1    4925 3375
-	-1   0    0    1
-$EndComp
-Wire Wire Line
-	3550 3075 3550 3375
-Wire Wire Line
-	4925 4275 4925 3975
-Wire Wire Line
-	4925 3075 4925 3375
-$Comp
-L power:+5V #PWR022
-U 1 1 5D490E86
-P 3550 3075
-F 0 "#PWR022" H 3550 2925 50  0001 C CNN
-F 1 "+5V" H 3565 3246 50  0000 C CNN
-F 2 "" H 3550 3075 50  0001 C CNN
-F 3 "" H 3550 3075 50  0001 C CNN
-	1    3550 3075
-	1    0    0    -1
-$EndComp
-$Comp
-L power:-12V #PWR024
-U 1 1 5D490AFD
-P 4925 4275
-F 0 "#PWR024" H 4925 4375 50  0001 C CNN
-F 1 "-12V" H 4940 4446 50  0000 C CNN
-F 2 "" H 4925 4275 50  0001 C CNN
-F 3 "" H 4925 4275 50  0001 C CNN
-	1    4925 4275
-	-1   0    0    1
-$EndComp
-$Comp
-L power:+12V #PWR023
-U 1 1 5D48FE4E
-P 4925 3075
-F 0 "#PWR023" H 4925 2925 50  0001 C CNN
-F 1 "+12V" H 4940 3246 50  0000 C CNN
-F 2 "" H 4925 3075 50  0001 C CNN
-F 3 "" H 4925 3075 50  0001 C CNN
-	1    4925 3075
-	1    0    0    -1
-$EndComp
 $EndSCHEMATC
