File: HW/IsolatedThreeOutputSMPS/ExternRegulatedConverters/18VIN_ExternRegulatedConverter_12D_12S_5S/ExternRegulatedConverter.sch (KiCad schematic (older format))
At the start: 27 parts, among them J1 15VDC, J2 Conn_01x07, U1 LM317L_SO8, U2 RS6-1205S, U3 RS6-1212D, U4 LM7812_TO220, U5 LM7812_TO220, U6 LM7912_TO220

Commit message: Update ExternRegulatedConverter.sch
Parts:
- removed D3, D4: 1N4001, symbol Device:D
- added D? (x2): ES2G, symbol Device:D
- D1: value D_Schottky -> BYS12-90-E3/TR
- D2: value 1N4001 -> ES2G
Changed lines of the file:
@@
 P 1925 1825
 F 0 "D1" H 1925 1609 50  0000 C CNN
-F 1 "D_Schottky" H 1925 1700 50  0000 C CNN
+F 1 "BYS12-90-E3/TR" H 1925 1700 50  0000 C CNN
 F 2 "Diode_SMD:D_SMA_Handsoldering" H 1925 1825 50  0001 C CNN
-F 3 "~" H 1925 1825 50  0001 C CNN
+F 3 "https://www.vishay.com/docs/88950/bys12-90.pdf" H 1925 1825 50  0001 C CNN
 	1    1925 1825
 	-1   0    0    1
@@
 P 3450 7250
 F 0 "D2" H 3450 7463 50  0000 C CNN
-F 1 "1N4001" H 3450 7374 50  0000 C CNN
+F 1 "ES2G" H 3450 7374 50  0000 C CNN
 F 2 "" H 3450 7250 50  0001 C CNN
-F 3 "~" H 3450 7250 50  0001 C CNN
+F 3 "https://www.vishay.com/docs/88588/es2f.pdf" H 3450 7250 50  0001 C CNN
 	1    3450 7250
 	1    0    0    -1
@@
 Wire Wire Line
 	4050 8000 4050 7725
-$Comp
-L Device:D D3
-U 1 1 5DA01D35
+Wire Wire Line
+	3450 8525 3450 8750
+Connection ~ 3450 8525
+Wire Wire Line
+	4050 8300 4050 8525
+Wire Wire Line
+	3450 8025 3450 8525
+Wire Wire Line
+	4050 8525 3450 8525
+Wire Wire Line
+	5900 8350 5900 7725
+Connection ~ 5900 7725
+Wire Wire Line
+	5900 7725 6325 7725
+Wire Wire Line
+	5900 8650 5900 9225
+Wire Wire Line
+	5900 9225 5375 9225
+Connection ~ 5375 9225
+$Comp
+L Device:D D?
+U 1 1 5D85587B
 P 4050 8150
-F 0 "D3" V 4005 8229 50  0000 L CNN
-F 1 "1N4001" V 4094 8229 50  0000 L CNN
+F 0 "D?" H 4050 8363 50  0000 C CNN
+F 1 "ES2G" H 4050 8274 50  0000 C CNN
 F 2 "" H 4050 8150 50  0001 C CNN
-F 3 "~" H 4050 8150 50  0001 C CNN
+F 3 "https://www.vishay.com/docs/88588/es2f.pdf" H 4050 8150 50  0001 C CNN
 	1    4050 8150
 	0    1    1    0
 $EndComp
-Wire Wire Line
-	3450 8525 3450 8750
-Connection ~ 3450 8525
-Wire Wire Line
-	4050 8300 4050 8525
-Wire Wire Line
-	3450 8025 3450 8525
-Wire Wire Line
-	4050 8525 3450 8525
-$Comp
-L Device:D D4
-U 1 1 5DA96FCE
+$Comp
+L Device:D D?
+U 1 1 5D8561FF
 P 5900 8500
-F 0 "D4" V 5855 8579 50  0000 L CNN
-F 1 "1N4001" V 5944 8579 50  0000 L CNN
+F 0 "D?" H 5900 8713 50  0000 C CNN
+F 1 "ES2G" H 5900 8624 50  0000 C CNN
 F 2 "" H 5900 8500 50  0001 C CNN
-F 3 "~" H 5900 8500 50  0001 C CNN
+F 3 "https://www.vishay.com/docs/88588/es2f.pdf" H 5900 8500 50  0001 C CNN
 	1    5900 8500
 	0    1    1    0
 $EndComp
-Wire Wire Line
-	5900 8350 5900 7725
-Connection ~ 5900 7725
-Wire Wire Line
-	5900 7725 6325 7725
-Wire Wire Line
-	5900 8650 5900 9225
-Wire Wire Line
-	5900 9225 5375 9225
-Connection ~ 5375 9225
 $EndSCHEMATC

Commit message: added 24V PSU
Parts:
- removed C5: 330nF, Capacitor_SMD:C_0805_2012Metric_Pad1.15x1.40mm_HandSolder, symbol Device:C
- removed C9: 10uF, symbol Device:CP
- removed D2, D?: ES2G, symbol Device:D
- removed R1: 2K7, symbol Device:R
- removed R2: 240R, symbol Device:R
- removed U1: LM317L_SO8, Package_SO:SOIC-8_3.9x4.9mm_P1.27mm, symbol Regulator_Linear:LM317L_SO8
- removed U5: LM7812_TO220, Package_TO_SOT_THT:TO-220-3_Vertical, symbol ExternRegulatedConverter-rescue:LM7812_TO220-Regulator_Linear
- added C10: 100nF, Capacitor_SMD:C_0805_2012Metric_Pad1.15x1.40mm_HandSolder, symbol Device:C
- added C13: 1uF, Capacitor_SMD:CP_Elec_4x5.7, symbol Device:CP
- added C9: 330nF, Capacitor_SMD:C_0805_2012Metric_Pad1.15x1.40mm_HandSolder, symbol Device:C
- added HS1: Heatsink 6.8K/W, Heatsink:Heatsink_SheetType_50x7mm_2Fixations, symbol Mechanical:Heatsink
- added U5: LM7805_TO220, Package_TO_SOT_THT:TO-220-3_Vertical, symbol Regulator_Linear:LM7805_TO220
- added U6: L7818CV, Package_TO_SOT_THT:TO-220-3_Vertical, symbol Regulator_Linear:LM7818_TO220
- added U7: L78M15ABV, Package_TO_SOT_THT:TO-220-3_Vertical, symbol Regulator_Linear:LM7815_TO220
- C5: renamed from C12; footprint (none) -> Capacitor_SMD:CP_Elec_4x5.7
- C6: value 100nF -> 330nF
- D2: renamed from D?; footprint (none) -> Diode_SMD:D_SMA_Handsoldering
- HS2: renamed from HS1; Mfr. No: (none) -> SK 480/50 SA; Mfr: (none) -> Fischer Elektronik; RSComponentsNo (none) -> 722-6874
- U1: renamed from U3; value RS6-1212D -> R2D-2415; footprint (none) -> RS6:RS6_DC_Converter
- U4: renamed from U2; value RS6-1205S -> ISE2409A-H; footprint (none) -> RS6:RS6_DC_Converter
- renumbered C10 to C11, C11 to C12, U4 to U2, U6 to U3
Connections:
- net labels added: +24V
- net labels removed: +18V, 12V
- wire segments 126 -> 119
Other:
- note added: "A) Analog PSU"
- note added: "B) Microcontroller PSU"
- note added: "C) Fan PSU"
- note added: "Inductive Load\nProtection"
- note added: "Input/Output Connectors"
- note added: "Pin Assignments:\n———————————\n1. Analog +12V\n2. Isolated GND\n3. Analog -12V\n4. Digital +5V\n5. Common GND\n6. Fan +15V\n7. Common GND\n\nPSU Module Nominal Current Usage: 65mA\n\nPSU Current Requirements:\n——————————————————\n\nA) Analog +/-12V —> CurrentSinkModule: 30mA\nB) Digital +5V —> ControlModule: 100mA\nC) +15V Fans —> Fans (x4): 150mA (700mA)"
- note added: "Shared Between Analog/MCU regulators"
- note added: "Thermal Spec:\n——————————\nAmb: 30C\n7818: 5K/W\n7815: 3K/W\nHS: 6.8K/W\n\nU6 JC Power Dissipation: (24V-18V) * 0.7A = 4.2W \nU6 JC Temp: 5 * 4.2 = 21 degC \n\nU7 JC Power Dissipation: (18V-15V) * 0.7A = 2.1W \nU7 JC Temp: 3 * 2.1 = 6.3 degC\n\nTotal Dissipation = 8.3W \nHS Temp = 8.3 * 6.8 = 56.5 degC\n\nTotal Temp = 30 + 21C + 6.3C + 56.5 = 113 degC"
- note added: "Unregulated"
- note removed: "1. Analog +12V\n2. Isolated GND\n3. Analog -12V\n4. Digital +5V\n5. Common GND\n6. Fan +15V\n7. Common GND"
- moved on the sheet: C1, C11, C12, C2, C3, C4, C5, C7, C8, D1, D2, HS2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

Commit message: RevA layout PSU
Parts:
- removed U1: R2D-2415, RS6:RS6_DC_Converter, symbol DCConverters:RS6-1212D
- removed U4: ISE2409A-H, RS6:RS6_DC_Converter, symbol DCConverters:RS6-1205S
- added C14: 4.7uF, Capacitor_SMD:CP_Elec_4x5.7, symbol Device:CP
- added U1: ISE2409A-H, XPower_Converter_DCDC:ISE, symbol DCConverters:ISE2409A-H
- added U4: R2D-2415, RS6:R2D, symbol DCConverters:R2D-2415
- C1: value 10uF -> 4.7uF
- C12: value 10uF -> 1uF
- C5: value 1uF -> 100nF
- C8: value 10uF -> 2.2uF
Connections:
- net +12V: no longer C3.1, C7.1, U2.1 (VI)
- net +15V: now also C3.1, C7.1, U2.1 (VI), U4.7 (+Vout)
- net +24V: now also C14.1, U1.2 (+Vin), U4.2 (+Vin)
- net -12V: no longer C4.1, C8.2, U3.2 (VI)
- net GNDS: now also C14.2, U1.1 (-Vin), U1.4 (0V), U4.1 (-Vin)
- net VCOM: now also U4.4 (COM)
- net +9V: now reaches C6.1, U5.1 (VI)
- net +9V: now also U1.5 (+Vout)
- net +18V: now reaches C5.1, C9.1, U6.3 (VO), U7.1 (VI)
- new net -15V: C4.1, C8.2, U3.2 (VI), U4.5 (-Vout)
- no-connect marks 5 -> 2
Other:
- moved on the sheet: C1, C11, C12, C3, C4, C7, C8, U2, U3

Commit message: updated RevA SMPS layout
Parts:
- added HS3: SK 481/50 SA, FischerElektronikHeatsinks:SK481_SK480_25MM, symbol Mechanical:Heatsink
- HS1: renamed from HS2; value Heatsink -> SK 480/50 SA; footprint Heatsink:Heatsink_SheetType_50x7mm_2Fixations -> FischerElektronikHeatsinks:SK512_SK480_50MM
- HS2: renamed from HS1; value Heatsink 6.8K/W -> SK 481/50 SA; footprint Heatsink:Heatsink_SheetType_50x7mm_2Fixations -> FischerElektronikHeatsinks:SK481_SK480_25MM; Mfr. No: SK 575/50 SA -> SK 481/50 SA; Type (none) -> 5.5K/W
- J1: footprint Connector_Molex:Molex_KK-254_AE-6410-02A_1x02_P2.54mm_Vertical -> Connector_PinHeader_2.54mm:PinHeader_1x02_P2.54mm_Horizontal
Connections:
- net +15V: now also J2.4 (Pin_4); no longer C3.1, C7.1, J2.6 (Pin_6), U2.1 (VI), U4.7 (+Vout)
- net +5V: now also J2.6 (Pin_6); no longer J2.4 (Pin_4)
- net -15V renamed -15VA
- new net +15VA: C3.1, C7.1, U2.1 (VI), U4.7 (+Vout)
Other:
- note added: "Pin Assignments:\n———————————\n1. Analog +12V\n2. Isolated GND\n3. Analog -12V\n4. Fan +15V\n5. Common GND\n6. Digital +5V\n7. Common GND\n\nPSU Module Nominal Current Usage: 65mA\n\nPSU Current Requirements:\n——————————————————\n\nA) Analog +/-12V —> CurrentSinkModule: 30mA\nB) Digital +5V —> ControlModule: 100mA\nC) +15V Fans —> Fans (x4): 150mA (700mA)"
- note added: "Thermal Spec:\n——————————\nAmb: 30C\n7818: 5K/W\n7815: 3K/W\nSK481: 5.5K/W\n"
- note added: "U6 JC Power Dissipation: (24V-18V) * 0.7A = 4.2W \nU6 JC Temp: 5 * 4.2 = 21 degC \n\nHS2 Temp = 4.2 * 5.5 = 23.1 degC\n\nTotal U6 Temp = 30 + 21C + 23.1 = 74 degC"
- note added: "U7 JC Power Dissipation: (18V-15V) * 0.7A = 2.1W \nU7 JC Temp: 3 * 2.1 = 6.3 degC\n \nHS3 Temp = 2.1 * 5.5 = 11.5 degC\n\nTotal U7 Temp = 30 + 6.3C + 11.5 = 47.8 degC"
- note removed: "Pin Assignments:\n———————————\n1. Analog +12V\n2. Isolated GND\n3. Analog -12V\n4. Digital +5V\n5. Common GND\n6. Fan +15V\n7. Common GND\n\nPSU Module Nominal Current Usage: 65mA\n\nPSU Current Requirements:\n——————————————————\n\nA) Analog +/-12V —> CurrentSinkModule: 30mA\nB) Digital +5V —> ControlModule: 100mA\nC) +15V Fans —> Fans (x4): 150mA (700mA)"
- note removed: "Thermal Spec:\n——————————\nAmb: 30C\n7818: 5K/W\n7815: 3K/W\nHS: 6.8K/W\n\nU6 JC Power Dissipation: (24V-18V) * 0.7A = 4.2W \nU6 JC Temp: 5 * 4.2 = 21 degC \n\nU7 JC Power Dissipation: (18V-15V) * 0.7A = 2.1W \nU7 JC Temp: 3 * 2.1 = 6.3 degC\n\nTotal Dissipation = 8.3W \nHS Temp = 8.3 * 6.8 = 56.5 degC\n\nTotal Temp = 30 + 21C + 6.3C + 56.5 = 113 degC"
- moved on the sheet: C13, C2, C5, C9, D2, HS2, U6, U7

Commit message: update
Parts:
- U2: symbol Regulator_Linear:LM7812_TO220 -> ExternRegulatedConverter-rescue:LM7812_TO220-Regulator_Linear
- U3: symbol Regulator_Linear:LM7912_TO220 -> ExternRegulatedConverter-rescue:LM7912_TO220-Regulator_Linear
- U5: symbol Regulator_Linear:LM7805_TO220 -> ExternRegulatedConverter-rescue:LM7805_TO220-Regulator_Linear
- U6: symbol Regulator_Linear:LM7818_TO220 -> ExternRegulatedConverter-rescue:LM7818_TO220-Regulator_Linear
- U7: symbol Regulator_Linear:LM7815_TO220 -> ExternRegulatedConverter-rescue:LM7815_TO220-Regulator_Linear
Changed lines of the file:
@@
 	5525 5875 5800 5875
 $Comp
-L Regulator_Linear:LM7812_TO220 U2
+L ExternRegulatedConverter-rescue:LM7812_TO220-Regulator_Linear U2
 U 1 1 5D8AD9F3
 P 7150 5175
@@
 $EndComp
 $Comp
-L Regulator_Linear:LM7912_TO220 U3
+L ExternRegulatedConverter-rescue:LM7912_TO220-Regulator_Linear U3
 U 1 1 5D8B3C95
 P 7150 6175
@@
 $EndComp
 $Comp
-L Regulator_Linear:LM7805_TO220 U5
+L ExternRegulatedConverter-rescue:LM7805_TO220-Regulator_Linear U5
 U 1 1 5D9569CB
 P 6825 8425
@@
 	10875 9750 1200 9750
 $Comp
-L Regulator_Linear:LM7818_TO220 U6
+L ExternRegulatedConverter-rescue:LM7818_TO220-Regulator_Linear U6
 U 1 1 5DB04640
 P 5175 12200
@@
 $EndComp
 $Comp
-L Regulator_Linear:LM7815_TO220 U7
+L ExternRegulatedConverter-rescue:LM7815_TO220-Regulator_Linear U7
 U 1 1 5DB0595F
 P 7750 12200
