File: HW/IsolatedThreeOutputSMPS/ExternRegulatedConverters/24VIN_ExternRegulatedConverter_12D_12S_5S/24VIN_ExternRegulatedConverter.sch (KiCad schematic (older format))
At the start: 28 parts, among them J1 15VDC, J2 Conn_01x07, U1 ISE2409A-H, U2 LM7812_TO220, U3 LM7912_TO220, U4 R2D-2415, U5 LM7805_TO220, U6 L7818CV, U7 L78M15ABV

Commit message: UPDATED 24VIN_PSU
- Added 5V  DC2DC input inductor (1mH)
- Added 3mm THT LEDs for output rail status
Parts:
- added D3, D4, D5, D6, D7: LED, LED_THT:LED_D3.0mm, symbol Device:LED
- added L1: 1mH, Inductor_SMD:L_Neosid_SM-NE127_HandSoldering, symbol pspice:INDUCTOR
- added R3: 10K, Resistor_SMD:R_1206_3216Metric_Pad1.42x1.75mm_HandSolder, symbol Device:R
- added R4: 6K8, Resistor_SMD:R_1206_3216Metric_Pad1.42x1.75mm_HandSolder, symbol Device:R
- added R5, R6: 4K7, Resistor_SMD:R_1206_3216Metric_Pad1.42x1.75mm_HandSolder, symbol Device:R
- added R7: 1K2, Resistor_SMD:R_1206_3216Metric_Pad1.42x1.75mm_HandSolder, symbol Device:R
- J1: value 15VDC -> 24VDC
- U2: symbol ExternRegulatedConverter-rescue:LM7812_TO220-Regulator_Linear -> 24VIN_ExternRegulatedConverter-rescue:LM7812_TO220-Regulator_Linear-ExternRegulatedConverter-rescue
- U3: symbol ExternRegulatedConverter-rescue:LM7912_TO220-Regulator_Linear -> 24VIN_ExternRegulatedConverter-rescue:LM7912_TO220-Regulator_Linear-ExternRegulatedConverter-rescue
- U5: symbol ExternRegulatedConverter-rescue:LM7805_TO220-Regulator_Linear -> 24VIN_ExternRegulatedConverter-rescue:LM7805_TO220-Regulator_Linear-ExternRegulatedConverter-rescue
- U6: symbol ExternRegulatedConverter-rescue:LM7818_TO220-Regulator_Linear -> 24VIN_ExternRegulatedConverter-rescue:LM7818_TO220-Regulator_Linear-ExternRegulatedConverter-rescue
- U7: symbol ExternRegulatedConverter-rescue:LM7815_TO220-Regulator_Linear -> 24VIN_ExternRegulatedConverter-rescue:LM7815_TO220-Regulator_Linear-ExternRegulatedConverter-rescue
Connections:
- wire segments 127 -> 143
Other:
- moved on the sheet: C13, C2, C5, C9, D2, HS2, HS3
