File: HW/IsolatedThreeOutputSMPS/ExternRegulatedConverters/24VIN_ExternRegulatedConverter_12D_24S_5S/24VIN_ExternRegulatedConverter_12D_24S_5S.kicad_pcb (KiCad board)
At the start: 2 copper layers, 69.8 x 44.5 mm, 32 parts, among them J1 24VDC, J2 Conn_01x07, Q1 IRF9540N, U1 L78L12_TO92, U2 L79L12_TO92, U4 R2D-2415, U5 LM7805_TO220

Commit message: updates
Parts:
- U1, U2: footprint Package_TO_SOT_THT:TO-92_Inline -> Package_TO_SOT_THT:TO-92_Inline_Wide
- moved D6 65.7 mm to (47.2, 73.7)
- moved C4 65.7 mm to (87.6, 80.0)
- moved C5 65.7 mm to (71.0, 70.0)
- moved R3 65.7 mm to (97.7, 63.8)
- moved C1 65.7 mm to (90.7, 58.9)
- moved C10 65.7 mm to (70.9, 94.2)
- moved C2 65.7 mm to (71.6, 60.2)
- moved C3 65.7 mm to (85.1, 58.2)
- moved C6 65.7 mm to (76.5, 94.2)
- moved C7 65.7 mm to (61.5, 61.5)
- moved C8 65.7 mm to (62.0, 71.1)
- moved D1 65.7 mm to (97.0, 86.9)
- moved D3 65.7 mm to (97.7, 57.0)
- moved R1 65.7 mm to (103.4, 86.9)
- moved REF** 65.7 mm to (43.7, 57.4)
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Connections:
- Q1 pad 2: +24V -> Net-(J1-Pad2)
- Q1 pad 3: Net-(J1-Pad2) -> +24V
Routing:
- net +24V: track 133.4 -> 129.8 mm, vias 1 -> 2
- net -12V: track 18.6 -> 20.0 mm
- net Net-(J1-Pad2): track 9.42 -> 8.64 mm
- net /-15VA: track 30.3 -> 30.9 mm
- net /+15VA: track 24.1 -> 24.6 mm
- net VCOM: track 0.00 -> 0.51 mm
