File: HW/ControlModule/Control.sch (KiCad schematic (older format))
At the start: 83 parts, among them U1 AD8629, U2 STM32L496VGTx, U3 LM4132AMF-3.3, U4 TLV70233DBVR

Commit message: updated HW
- Added front panel NRST switch
- Changed 0402 to 0805 input filter, added NC jumper
Parts:
- C1, C2, C26, C27, C3, C4: footprint Capacitor_SMD:C_0402_1005Metric -> Capacitor_SMD:C_0805_2012Metric_Pad1.15x1.40mm_HandSolder
- JP5, JP6: footprint Jumper:SolderJumper-2_P1.3mm_Open_Pad1.0x1.5mm -> Jumper:SolderJumper-2_P1.3mm_Bridged_Pad1.0x1.5mm
- R1, R2, R3, R4, R8, R9: footprint Resistor_SMD:R_0402_1005Metric -> Resistor_SMD:R_0805_2012Metric_Pad1.15x1.40mm_HandSolder
Changed lines of the file:
@@
 F 0 "R3" V 3543 3150 50  0000 C CNN
 F 1 "100R" V 3634 3150 50  0000 C CNN
-F 2 "Resistor_SMD:R_0402_1005Metric" V 3680 3150 50  0001 C CNN
+F 2 "Resistor_SMD:R_0805_2012Metric_Pad1.15x1.40mm_HandSolder" V 3680 3150 50  0001 C CNN
 F 3 "~" H 3750 3150 50  0001 C CNN
 	1    3750 3150
@@
 F 0 "C3" V 5000 2600 50  0000 L CNN
 F 1 "0F" V 4900 2600 50  0000 L CNN
-F 2 "Capacitor_SMD:C_0402_1005Metric" H 4788 2500 50  0001 C CNN
+F 2 "Capacitor_SMD:C_0805_2012Metric_Pad1.15x1.40mm_HandSolder" H 4788 2500 50  0001 C CNN
 F 3 "~" H 4750 2650 50  0001 C CNN
 	1    4750 2650
@@
 F 0 "R1" V 2993 5950 50  0000 C CNN
 F 1 "0R" V 3084 5950 50  0000 C CNN
-F 2 "Resistor_SMD:R_0402_1005Metric" V 3130 5950 50  0001 C CNN
+F 2 "Resistor_SMD:R_0805_2012Metric_Pad1.15x1.40mm_HandSolder" V 3130 5950 50  0001 C CNN
 F 3 "~" H 3200 5950 50  0001 C CNN
 	1    3200 5950
@@
 F 0 "C4" V 4500 5300 50  0000 L CNN
 F 1 "0F" V 4600 5350 50  0000 L CNN
-F 2 "Capacitor_SMD:C_0402_1005Metric" H 4788 5200 50  0001 C CNN
+F 2 "Capacitor_SMD:C_0805_2012Metric_Pad1.15x1.40mm_HandSolder" H 4788 5200 50  0001 C CNN
 F 3 "~" H 4750 5350 50  0001 C CNN
 	1    4750 5350
@@
 F 0 "C1" H 3900 3550 50  0000 L CNN
 F 1 "100nF" H 3900 3450 50  0000 L CNN
-F 2 "Capacitor_SMD:C_0402_1005Metric" H 4138 3350 50  0001 C CNN
+F 2 "Capacitor_SMD:C_0805_2012Metric_Pad1.15x1.40mm_HandSolder" H 4138 3350 50  0001 C CNN
 F 3 "~" H 4100 3500 50  0001 C CNN
 	1    4100 3500
@@
 F 0 "R2" V 3043 3150 50  0000 C CNN
 F 1 "0R" V 3134 3150 50  0000 C CNN
-F 2 "Resistor_SMD:R_0402_1005Metric" V 3180 3150 50  0001 C CNN
+F 2 "Resistor_SMD:R_0805_2012Metric_Pad1.15x1.40mm_HandSolder" V 3180 3150 50  0001 C CNN
 F 3 "~" H 3250 3150 50  0001 C CNN
 	1    3250 3150
@@
 F 0 "R4" V 3543 5950 50  0000 C CNN
 F 1 "100R" V 3634 5950 50  0000 C CNN
-F 2 "Resistor_SMD:R_0402_1005Metric" V 3680 5950 50  0001 C CNN
+F 2 "Resistor_SMD:R_0805_2012Metric_Pad1.15x1.40mm_HandSolder" V 3680 5950 50  0001 C CNN
 F 3 "~" H 3750 5950 50  0001 C CNN
 	1    3750 5950
@@
 F 0 "C2" H 4215 6346 50  0000 L CNN
 F 1 "100nF" H 4215 6255 50  0000 L CNN
-F 2 "Capacitor_SMD:C_0402_1005Metric" H 4138 6150 50  0001 C CNN
+F 2 "Capacitor_SMD:C_0805_2012Metric_Pad1.15x1.40mm_HandSolder" H 4138 6150 50  0001 C CNN
 F 3 "~" H 4100 6300 50  0001 C CNN
 	1    4100 6300
@@
 F 0 "R8" V 5125 3600 50  0000 C CNN
 F 1 "0R" V 5125 3950 50  0000 C CNN
-F 2 "Resistor_SMD:R_0402_1005Metric" V 5180 3800 50  0001 C CNN
+F 2 "Resistor_SMD:R_0805_2012Metric_Pad1.15x1.40mm_HandSolder" V 5180 3800 50  0001 C CNN
 F 3 "~" H 5250 3800 50  0001 C CNN
 	1    5250 3800
@@
 F 0 "C26" V 5050 4100 50  0000 L CNN
 F 1 "0F" V 5050 3800 50  0000 L CNN
-F 2 "Capacitor_SMD:C_0402_1005Metric" H 5288 3850 50  0001 C CNN
+F 2 "Capacitor_SMD:C_0805_2012Metric_Pad1.15x1.40mm_HandSolder" H 5288 3850 50  0001 C CNN
 F 3 "~" H 5250 4000 50  0001 C CNN
 	1    5250 4000
@@
 F 0 "R9" V 5125 6400 50  0000 C CNN
 F 1 "0R" V 5125 6750 50  0000 C CNN
-F 2 "Resistor_SMD:R_0402_1005Metric" V 5180 6600 50  0001 C CNN
+F 2 "Resistor_SMD:R_0805_2012Metric_Pad1.15x1.40mm_HandSolder" V 5180 6600 50  0001 C CNN
 F 3 "~" H 5250 6600 50  0001 C CNN
 	1    5250 6600
@@
 F 0 "C27" V 5050 6900 50  0000 L CNN
 F 1 "oF" V 5050 6550 50  0000 L CNN
-F 2 "Capacitor_SMD:C_0402_1005Metric" H 5288 6650 50  0001 C CNN
+F 2 "Capacitor_SMD:C_0805_2012Metric_Pad1.15x1.40mm_HandSolder" H 5288 6650 50  0001 C CNN
 F 3 "~" H 5250 6800 50  0001 C CNN
 	1    5250 6800
@@
 F 0 "JP5" H 5200 4731 50  0000 C CNN
 F 1 "BYPASS" H 5200 4642 50  0000 C CNN
-F 2 "Jumper:SolderJumper-2_P1.3mm_Open_Pad1.0x1.5mm" H 5200 4550 50  0001 C CNN
+F 2 "Jumper:SolderJumper-2_P1.3mm_Bridged_Pad1.0x1.5mm" H 5200 4550 50  0001 C CNN
 F 3 "~" H 5200 4550 50  0001 C CNN
 	1    5200 4550
@@
 F 0 "JP6" H 5200 7581 50  0000 C CNN
 F 1 "BYPASS" H 5200 7492 50  0000 C CNN
-F 2 "Jumper:SolderJumper-2_P1.3mm_Open_Pad1.0x1.5mm" H 5200 7400 50  0001 C CNN
+F 2 "Jumper:SolderJumper-2_P1.3mm_Bridged_Pad1.0x1.5mm" H 5200 7400 50  0001 C CNN
 F 3 "~" H 5200 7400 50  0001 C CNN
 	1    5200 7400
